File: hardware/rev-e/kicad/PSN-Presepe-Mega-RevE.kicad_pcb (KiCad board)
At the start: 2 copper layers, 300 x 180 mm, 104 parts, among them J1 12V_IN, K1 G5Q-1_DC12, K10 G5Q-1_DC12, K11 G5Q-1_DC12, K12 G5Q-1_DC12, K13 G5Q-1_DC12, K14 G5Q-1_DC12, K15 G5Q-1_DC12, K16 G5Q-1_DC12, K2 G5Q-1_DC12, K3 G5Q-1_DC12, K4 G5Q-1_DC12, K5 G5Q-1_DC12, K6 G5Q-1_DC12, K7 G5Q-1_DC12, K8 G5Q-1_DC12, K9 G5Q-1_DC12, Q1 IRLZ44N_CIELO_R, Q2 IRLZ44N_CIELO_G, Q3 IRLZ44N_CIELO_B, Q4 IRLZ44N_TRAM_R, Q5 IRLZ44N_TRAM_G, Q6 IRLZ44N_TRAM_B, Q7 IRLZ44N_ALBA_R, Q8 IRLZ44N_ALBA_G, Q9 IRLZ44N_ALBA_B, U1 ULN2803A, U2 ULN2803A, U3 AMS1117-3.3, U4 74LVC125A

Commit message: Rev E: fixes from the independent review
- Test points now TP1-TP5 in the order 12V, GND, 5V, GND, 3V3: a slipping
  probe can only short a rail to GND (never 12 V onto the Mega's 5 V or
  5 V onto the 3.3 V of the microSD); verify.py checks the order.
- USB no-via rule area is now also in the routed board, so KiCad DRC keeps
  enforcing it after any later edit.
- Copper sliver fix in cleanup.py (only when DRC reports one): fill the
  seam of same-net tangent tracks and bridge track ends that just touch a
  same-net track; deterministic output, net-class widths respected.
- Assembly PDF counts SMD parts from the board (12); TP symbols not in the
  schematic BOM; Gerber checker uses 0.25 mm for +5V like the board check.
- New routing session; replaying it gives identical Gerbers. DRC 0,
  independent checks pass, min spacing 0.222 mm. README updated.

Co-Authored-By: Claude Opus 5.5 <noreply@anthropic.com>
Claude-Session: https://claude.ai/code/session_01S57jeHAWREhchCq9pZcfbq
Parts:
- added TP5: TP_GND, TestPoint_THTPad_D2.0mm_Drill1.0mm, F.Cu at (46.5, 33.5)
- moved TP3 10.0 mm to (51.5, 33.5)
- moved TP4 10.0 mm to (36.5, 33.5)
- moved TP2 5.00 mm to (41.5, 33.5)
- moved D1 4.00 mm to (56.5, 29.0)
- moved RLED 3.50 mm to (63.5, 29.0)
Routing:
- net ALBA_G_NEG: track 161.0 -> 105.1 mm
- net D20_SDA: track 209.2 -> 179.3 mm, vias 3 -> 0
- net D44_ALBA_R: track 180.0 -> 152.4 mm, vias 1 -> 3
- net CIELO_G_NEG: track 91.1 -> 116.7 mm, vias 1 -> 2
- net D23_NEXT: track 194.9 -> 172.5 mm, vias 1 -> 0
- net +3V3: track 128.7 -> 108.0 mm, vias 3 -> 1
- net D21_SCL: track 206.0 -> 186.2 mm, vias 4 -> 1
- net GND: track 956.0 -> 974.5 mm
- net D52_SD_SCK: track 67.0 -> 85.4 mm, vias 1 -> 2
- net RELAY9_COIL_LOW: track 194.4 -> 177.2 mm, vias 1 -> 0
- net D5_STELLE_DATA: track 216.3 -> 233.3 mm, vias 0 -> 1
- net D8_CASETTE_DATA: track 265.2 -> 249.1 mm
- net D22_START: track 190.4 -> 174.7 mm, vias 4 -> 0
- net ALBA_B_NEG: track 97.6 -> 82.2 mm, vias 1 -> 0
- net TRAM_B_NEG: track 81.5 -> 67.6 mm
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