File: hardware/rev-e/kicad/PSN-Presepe-Mega-RevE.kicad_sch (KiCad schematic)
At the start: 95 parts, among them J1 12V_IN, K1 G5Q-1_DC12, K10 G5Q-1_DC12, K11 G5Q-1_DC12, K12 G5Q-1_DC12, K13 G5Q-1_DC12, K14 G5Q-1_DC12, K15 G5Q-1_DC12, K16 G5Q-1_DC12, K2 G5Q-1_DC12, K3 G5Q-1_DC12, K4 G5Q-1_DC12, K5 G5Q-1_DC12, K6 G5Q-1_DC12, K7 G5Q-1_DC12, K8 G5Q-1_DC12, K9 G5Q-1_DC12, Q1 IRLZ44N_CIELO_R, Q2 IRLZ44N_CIELO_G, Q3 IRLZ44N_CIELO_B, Q4 IRLZ44N_TRAM_R, Q5 IRLZ44N_TRAM_G, Q6 IRLZ44N_TRAM_B, Q7 IRLZ44N_ALBA_R, Q8 IRLZ44N_ALBA_G, Q9 IRLZ44N_ALBA_B, U1 ULN2803A, U2 ULN2803A, U3 AMS1117-3.3, U4 74LVC125A

Commit message: Rev E: fixes from the independent review
- Test points now TP1-TP5 in the order 12V, GND, 5V, GND, 3V3: a slipping
  probe can only short a rail to GND (never 12 V onto the Mega's 5 V or
  5 V onto the 3.3 V of the microSD); verify.py checks the order.
- USB no-via rule area is now also in the routed board, so KiCad DRC keeps
  enforcing it after any later edit.
- Copper sliver fix in cleanup.py (only when DRC reports one): fill the
  seam of same-net tangent tracks and bridge track ends that just touch a
  same-net track; deterministic output, net-class widths respected.
- Assembly PDF counts SMD parts from the board (12); TP symbols not in the
  schematic BOM; Gerber checker uses 0.25 mm for +5V like the board check.
- New routing session; replaying it gives identical Gerbers. DRC 0,
  independent checks pass, min spacing 0.222 mm. README updated.

Co-Authored-By: Claude Opus 5.5 <noreply@anthropic.com>
Claude-Session: https://claude.ai/code/session_01S57jeHAWREhchCq9pZcfbq
Parts:
- added TP5: TP_GND, TestPoint_THTPad_D2.0mm_Drill1.0mm, symbol PSN:TP5
- TP1, TP2, TP3, TP4: now left out of the parts list
Connections:
- net GND: now also TP5.1 (GND)
